Commit message: modified urdf and added some gazebo tags

File: diff_drive/urdf/ddrive.urdf.xacro (robot description, xacro)
@@ -1,7 +1,13 @@
 <robot name="buttercup" xmlns:xacro="http://www.ros.org/wiki/xacro">
+<xacro:include filename="$(find diff_drive)/ddrive.gazebo.xacro"/>
+<xacro:property name="params_yaml" value="$(find diff_drive)/robot_params.yaml"/>
+<xacro:property name="yaml_dict" value="${xacro.load_yaml(params_yaml)}"/>
+<xacro:property name="chassis_core" value="${yaml_dict['robot_params']['chassis_core']}"/>
+<xacro:property name="wheel_radius" value="${yaml_dict['robot_params']['wheel_radius']}"/>
+<xacro:property name="caster_radius" value="${yaml_dict['robot_params']['caster_radius']}"/>
 <link name="base_link">
     <visual>
         <geometry>
-            <box size="1.5 1.0 0.25"/>
+            <box size="${chassis_core*2} ${chassis_core} ${chassis_core*0.5}"/>
         </geometry>
         <material name="red_mat">
@@ -11,5 +17,5 @@
     <collision>
        <geometry>
-            <box size="2.0 1.0 0.5"/>
+            <box size="${chassis_core*1.5} ${chassis_core} ${chassis_core*0.25}"/>
         </geometry>
         <material name="red_mat">
@@ -21,5 +27,5 @@
     <visual>
         <geometry>
-            <sphere radius="0.2"/>
+            <sphere radius="${caster_radius}"/>
         </geometry>
         <material name="green_mat">
@@ -29,5 +35,5 @@
     <collision>
         <geometry>
-            <sphere radius="0.2"/>
+            <sphere radius="${caster_radius}"/>
         </geometry>
         <material name="green_mat">
@@ -39,5 +45,5 @@
     <visual>
         <geometry>
-            <sphere radius="0.2"/>
+            <sphere radius="${caster_radius}"/>
         </geometry>
         <material name="green_mat">
@@ -47,5 +53,5 @@
     <collision>
         <geometry>
-            <sphere radius="0.2"/>
+            <sphere radius="${caster_radius}"/>
         </geometry>
         <material name="green_mat">
@@ -57,5 +63,5 @@
     <visual>
         <geometry>
-            <cylinder radius="0.3" length="0.2"/>
+            <cylinder radius="${wheel_radius}" length="0.2"/>
         </geometry>
         <material name="blue_mat">
@@ -65,5 +71,5 @@
     <collision>
         <geometry>
-            <cylinder radius="0.3" length="0.2"/>
+            <cylinder radius="${wheel_radius}" length="0.2"/>
         </geometry>
         <material name="blue_mat">
@@ -75,5 +81,5 @@
     <visual>
         <geometry>
-            <cylinder radius="0.3" length="0.2"/>
+            <cylinder radius="${wheel_radius}" length="0.2"/>
         </geometry>
         <material name="blue_mat">
@@ -83,5 +89,5 @@
     <collision>
         <geometry>
-            <cylinder radius="0.3" length="0.2"/>
+            <cylinder radius="${wheel_radius}" length="0.2"/>
         </geometry>
         <material name="blue_mat">
@@ -91,5 +97,5 @@
 </link>
 <joint name="bottom_caster_wheel" type="continuous">
-    <origin xyz="0.5 0 -0.125" rpy="0 0 0"/>
+    <origin xyz="${chassis_core*2*0.4} 0 -${chassis_core*0.5*0.5}" rpy="0 0 0"/>
     <parent link="base_link"/>
     <child link="bottom_caster"/>
@@ -97,5 +103,5 @@
 </joint>
 <joint name="top_caster_wheel" type="continuous">
-    <origin xyz="0.5 0 0.125" rpy="0 0 0"/>
+    <origin xyz="${chassis_core*2*0.4} 0 ${chassis_core*0.5*0.5}" rpy="0 0 0"/>
     <parent link="base_link"/>
     <child link="top_caster"/>
@@ -103,5 +109,5 @@
 </joint>
 <joint name="left_wheel_base" type="continuous">
-    <origin xyz="-0.5 0.6 0" rpy="-1.57 0 0"/>
+    <origin xyz="-${chassis_core*0.5} 0.6 0" rpy="-1.57 0 0"/>
     <parent link="base_link"/>
     <child link="left_wheel"/>
@@ -109,5 +115,5 @@
 </joint>
 <joint name="right_wheel_base" type="continuous">
-    <origin xyz="-0.5 -0.6 0" rpy="1.57 0 0"/>
+    <origin xyz="-${chassis_core*0.5} -0.6 0" rpy="1.57 0 0"/>
     <parent link="base_link"/>
     <child link="right_wheel"/>
