Commit message: Spawned model in gazebo, set up ros gz bridge, added rviz config

File: diff_drive/urdf/ddrive.gazebo.xacro (robot description, xacro)
@@ -1,32 +1,14 @@
 <robot name="buttercup" xmlns:xacro="http://www.ros.org/wiki/xacro">
-<gazebo reference="base_link">
-     <inertial>
-        <mass value="1.14395"/>
-        <inertia ixx="0.095329" iyy="0.381317" izz="0.476646"/>
-    </inertial>
-</gazebo>
-<gazebo reference="left_wheel">
-<inertial>
-        <mass value="1"/>
-        <inertia ixx="0.043333" iyy="0.043333" izz="0.08"/>
-    </inertial>
-</gazebo>
-<gazebo reference="right_wheel">
- <inertial>
-        <mass value="1"/>
-        <inertia ixx="0.043333" iyy="0.043333" izz="0.08"/>
-    </inertial>
-</gazebo>
-<gazebo reference="top_caster">
- <inertial>
-        <mass value="1"/>
-        <inertia ixx="0.016" iyy="0.016" izz="0.016"/>
-    </inertial>
-</gazebo>
-<gazebo reference="bottom_caster">
-<inertial>
-    <mass value="1"/>
-        <inertia ixx="0.016" iyy="0.016" izz="0.016"/>
-    </inertial>
+<gazebo >
+    <plugin filename="libgz-sim-diff-drive-system.so" name="gz::sim::systems::DiffDrive">
+        <left_joint>left_wheel_base</left_joint>
+        <right_joint>right_wheel_base</right_joint>
+        <wheel_separation>1.2</wheel_separation>
+        <wheel_radius>0.4</wheel_radius>
+        <odom_publish_frequency>1</odom_publish_frequency>
+        <topic>cmd_vel</topic>
+    </plugin>
+    <plugin filename="libgz-sim-joint-state-publisher-system.so" name="gz::sim::systems::JointStatePublisher">
+    </plugin>
 </gazebo>
 </robot>

File: diff_drive/urdf/ddrive.urdf.xacro (robot description, xacro)
@@ -1,4 +1,3 @@
 <robot name="buttercup" xmlns:xacro="http://www.ros.org/wiki/xacro">
-<xacro:include filename="$(find diff_drive)/ddrive.gazebo.xacro"/>
 <xacro:property name="params_yaml" value="$(find diff_drive)/robot_params.yaml"/>
 <xacro:property name="yaml_dict" value="${xacro.load_yaml(params_yaml)}"/>
@@ -23,4 +22,8 @@
         </material>
     </collision>
+    <inertial>
+        <mass value="1.14395"/>
+        <inertia ixx="0.095329" iyy="0.381317" ixy="0.0" ixz="0.0" iyz="0.0" izz="0.476646"/>
+    </inertial>
 </link>
 <link name="bottom_caster">
@@ -41,4 +44,8 @@
         </material>
     </collision>
+    <inertial>
+        <mass value="1"/>
+        <inertia ixx="0.016" ixy="0.0" ixz="0.0" iyy="0.016" iyz="0.0" izz="0.016"/>
+    </inertial>
 </link>
 <link name="top_caster">
@@ -59,4 +66,8 @@
         </material>
     </collision>
+    <inertial>
+        <mass value="1"/>
+        <inertia ixx="0.016" ixy="0.0" ixz="0.0" iyy="0.016" iyz="0.0" izz="0.016"/>
+    </inertial>
 </link>
 <link name="left_wheel">
@@ -77,4 +88,8 @@
         </material>
     </collision>
+    <inertial>
+        <mass value="1"/>
+        <inertia ixx="0.043333" ixy="0.0" ixz="0.0" iyy="0.043333" iyz="0.0" izz="0.08"/>
+    </inertial>
 </link>
 <link name="right_wheel">
@@ -95,4 +110,8 @@
         </material>
     </collision>
+   <inertial>
+        <mass value="1"/>
+        <inertia ixx="0.043333" ixy="0.0" ixz="0.0" iyy="0.043333" iyz="0.0" izz="0.08"/>
+    </inertial>
 </link>
 <joint name="bottom_caster_wheel" type="continuous">
@@ -120,3 +139,4 @@
     <axis xyz="0 0 1"/>
 </joint>
+<xacro:include filename="$(find diff_drive)/ddrive.gazebo.xacro"/>
 </robot>

Commit message: Added flip node and xml launch files

File: diff_drive/urdf/ddrive.gazebo.xacro (robot description, xacro)
@@ -1,3 +1,19 @@
 <robot name="buttercup" xmlns:xacro="http://www.ros.org/wiki/xacro">
+<gazebo reference="top_caster">
+    <mu1>0.0</mu1>
+    <mu2>0.0</mu2>
+</gazebo>
+<gazebo reference="bottom_caster">
+    <mu1>0.0</mu1>
+    <mu2>0.0</mu2>
+</gazebo>
+<gazebo reference="left_wheel">
+    <mu1>10000.0</mu1>
+    <mu2>10000.0</mu2>
+</gazebo>
+<gazebo reference="right_wheel">
+    <mu1>10000.0</mu1>
+    <mu2>10000.0</mu2>
+</gazebo>
 <gazebo >
     <plugin filename="libgz-sim-diff-drive-system.so" name="gz::sim::systems::DiffDrive">

File: diff_drive/urdf/ddrive.urdf.xacro (robot description, xacro)
@@ -16,5 +16,5 @@
     <collision>
        <geometry>
-            <box size="${chassis_core*1.5} ${chassis_core} ${chassis_core*0.25}"/>
+            <box size="${chassis_core*2} ${chassis_core} ${chassis_core*0.5}"/>
         </geometry>
         <material name="red_mat">
@@ -23,6 +23,6 @@
     </collision>
     <inertial>
-        <mass value="1.14395"/>
-        <inertia ixx="0.095329" iyy="0.381317" ixy="0.0" ixz="0.0" iyz="0.0" izz="0.476646"/>
+        <mass value="2.0"/>
+        <inertia ixx="1.0" iyy="1.0" ixy="0.0" ixz="0.0" iyz="0.0" izz="1.0"/>
     </inertial>
 </link>
@@ -45,6 +45,6 @@
     </collision>
     <inertial>
-        <mass value="1"/>
-        <inertia ixx="0.016" ixy="0.0" ixz="0.0" iyy="0.016" iyz="0.0" izz="0.016"/>
+        <mass value="2.0"/>
+        <inertia ixx="0.032" ixy="0.0" ixz="0.0" iyy="0.032" iyz="0.0" izz="0.032"/>
     </inertial>
 </link>
@@ -67,10 +67,11 @@
     </collision>
     <inertial>
-        <mass value="1"/>
-        <inertia ixx="0.016" ixy="0.0" ixz="0.0" iyy="0.016" iyz="0.0" izz="0.016"/>
+        <mass value="2.0"/>
+        <inertia ixx="0.032" ixy="0.0" ixz="0.0" iyy="0.032" iyz="0.0" izz="0.032"/>
     </inertial>
 </link>
 <link name="left_wheel">
     <visual>
+        <origin xyz="0 0 0" rpy="1.57 0 0"/>
         <geometry>
             <cylinder radius="${wheel_radius}" length="0.2"/>
@@ -81,4 +82,5 @@
     </visual>
     <collision>
+        <origin xyz="0 0 0" rpy="1.57 0 0"/>
         <geometry>
             <cylinder radius="${wheel_radius}" length="0.2"/>
@@ -89,10 +91,12 @@
     </collision>
     <inertial>
-        <mass value="1"/>
-        <inertia ixx="0.043333" ixy="0.0" ixz="0.0" iyy="0.043333" iyz="0.0" izz="0.08"/>
+        <origin xyz="0 0 0" rpy="1.57 0 0"/>
+        <mass value="20.0"/>
+        <inertia ixx="1.0" ixy="0.0" ixz="0.0" iyy="1.0" iyz="0.0" izz="1.0"/>
     </inertial>
 </link>
 <link name="right_wheel">
     <visual>
+        <origin xyz="0 0 0" rpy="1.57 0 0"/>
         <geometry>
             <cylinder radius="${wheel_radius}" length="0.2"/>
@@ -103,4 +107,5 @@
     </visual>
     <collision>
+        <origin xyz="0 0 0" rpy="1.57 0 0"/>
         <geometry>
             <cylinder radius="${wheel_radius}" length="0.2"/>
@@ -111,31 +116,32 @@
     </collision>
    <inertial>
-        <mass value="1"/>
-        <inertia ixx="0.043333" ixy="0.0" ixz="0.0" iyy="0.043333" iyz="0.0" izz="0.08"/>
+        <origin xyz="0 0 0" rpy="1.57 0 0"/>
+        <mass value="20.0"/>
+        <inertia ixx="1.0" ixy="0.0" ixz="0.0" iyy="1.0" iyz="0.0" izz="1.0"/>
     </inertial>
 </link>
-<joint name="bottom_caster_wheel" type="continuous">
-    <origin xyz="${chassis_core*2*0.4} 0 -${chassis_core*0.5*0.5}" rpy="0 0 0"/>
+<joint name="bottom_caster_wheel" type="fixed">
+    <origin xyz="-${chassis_core*2*0.4} 0 -${chassis_core*0.5*0.5}" rpy="0 0 0"/>
     <parent link="base_link"/>
     <child link="bottom_caster"/>
-    <axis xyz="1 1 1"/>
+    <!-- <axis xyz="1 1 1"/> -->
 </joint>
-<joint name="top_caster_wheel" type="continuous">
-    <origin xyz="${chassis_core*2*0.4} 0 ${chassis_core*0.5*0.5}" rpy="0 0 0"/>
+<joint name="top_caster_wheel" type="fixed">
+    <origin xyz="-${chassis_core*2*0.4} 0 ${chassis_core*0.5*0.5}" rpy="0 0 0"/>
     <parent link="base_link"/>
     <child link="top_caster"/>
-    <axis xyz="1 1 1"/>
+    <!-- <axis xyz="1 1 1"/> -->
 </joint>
 <joint name="left_wheel_base" type="continuous">
-    <origin xyz="-${chassis_core*0.5} 0.6 0" rpy="-1.57 0 0"/>
+    <origin xyz="${chassis_core*0.9} 0.6 0" rpy="0 0 0"/>
     <parent link="base_link"/>
     <child link="left_wheel"/>
-    <axis xyz="0 0 1"/>
+    <axis xyz="0 1 0"/>
 </joint>
 <joint name="right_wheel_base" type="continuous">
-    <origin xyz="-${chassis_core*0.5} -0.6 0" rpy="1.57 0 0"/>
+    <origin xyz="${chassis_core*0.9} -0.6 0" rpy="0 0 0"/>
     <parent link="base_link"/>
     <child link="right_wheel"/>
-    <axis xyz="0 0 1"/>
+    <axis xyz="0 1 0"/>
 </joint>
 <xacro:include filename="$(find diff_drive)/ddrive.gazebo.xacro"/>
